File: PHONE2.brd (EAGLE design)
At the start: 127 x 53.3 mm, 106 parts, among them IC1 ATMEGA1284P, IC2 FT230X, IC3 LTC4054, IC4 LP2985-33DBVR, J1 Power, J2 Analog, J3 Digital_8_13, J4 Digital_0_7, P1 USB-6PSMT, P2 ICSP:MAIN, Q1 2N7002 SOT-23, Q2 2N7002, Q3 BC846ALTIG, SW0 0, SW1 1, SW10 *, SW11 #, SW12 LEFT, SW13 DOWN, SW14 RIGHT, SW15 UP, SW2 2, SW3 3, SW4 4, SW5 5, SW6 6, SW7 7, SW8 8, SW9 9, X1 8MHz

Commit message: Routing and schematic work
Parts:
- removed C2, C3: 22pF 0603, freetronics-master-v1.1:0603
- removed Q3: BC846ALTIG, freetronics-original:SOT23-3
- removed R18: 10K 0603, freetronics-master-v1.1:0603
- removed S5: Hirose DF12C(3.0)-50DP-0.5V, freetronics-jon:ADH8066
- removed TP3, TP4, TP5: TEST-POINT, freetronics-original:PAD.02X.02
- removed X1: 8MHz, freetronics-master-v1:HC49U-V
- added C18, C20, C21: 100nF, freetronics-master-v1:0603
- added C19: 22pF, freetronics-master-v1:0603
- added IC5: SIM900, ICs_v54:SIM900
- added J6: SIM Socket, SparkFun2:SIMHOLDER3
- added Q4: 2N7002, freetronics-luke:SOT23-3
- added R22, R23, R24: 22R, freetronics-master-v1:0603
- added R25: 100K, freetronics-master-v1:0603
- added R26: 10R, freetronics-master-v1:0603
- added U$9: XH414H-IV01E, cellphone:414-VA5R
- added Y1: RESONATORSMD, SparkFun:RESONATOR-SMD
- added Z1, Z2: PGB102ST23, freetronics-luke:SOT23-3
- R6: value 1M 0603 -> 100K; device freetronics-master-v1.1:0603 -> freetronics-master-v1:0603
- TP1, TP2: value TEST-POINT -> TEST-POINT2
- moved TP2 32.6 mm to (53.3, 30.2)
- moved TP1 32.5 mm to (53.6, 28.4)
- moved R8 30.8 mm to (42.4, 43.2), turned to 180 degrees
- moved R6 30.2 mm to (32.3, 41.7)
- moved R9 24.9 mm to (42.4, 40.6), turned to 180 degrees
Connections:
- removed net N$20: JP13.1, S4.3, S4.4, S5.49
- removed net N$21: R8.2, S5.15
- removed net N$22: R9.2, S5.17
- removed net N$23: S5.18, TP3.P$1
- removed net N$24: S5.19, TP4.P$1
- removed net N$25: S5.20, TP5.P$1
- removed net N$26: R18.2, S5.31
- removed net N$30: S5.11, TP1.P$1
- removed net N$31: S5.12, TP2.P$1
- removed net XTL1: C3.2, IC1.8, R6.1, X1.1
- removed net XTL2: C2.2, IC1.7, R6.2, X1.2
- new net !GSM_RESET: C18.2, IC5.16
- new net CTS: IC5.7
- new net DBG_RXD: IC5.28, TP1.P$1
- new net DBG_TXD: IC5.27, TP2.P$1
- new net DCD: IC5.5
- new net DISP_CLK: IC5.11
- new net DISP_CS: IC5.14
- new net DISP_DATA: IC5.12
- new net DISP_DC: IC5.13
- new net EARN: JP13.2, S4.1, SJ6.1
- new net EARP: JP13.1, S4.3, S4.4
- new net MIC+: IC5.19
- new net MIC-: IC5.20
- new net MIC1N: SJ3.2, SJ6.2
- new net MIC1P: S4.2A, S4.2B, SJ2.2
- new net N$28: J6.2, R23.2, Z2.1
- new net N$29: IC5.26, U$9.+
- new net N$40: J6.3, R22.2, Z1.1
- new net N$49: J6.4, R24.2, Z1.2
- new net N$69: Q4.1, R25.2, R26.1
- new net NETWORK_LED: IC5.52
- new net RF_ANT: IC5.60
- new net RI: IC5.4
- new net RTS: IC5.8
- new net RXD: IC5.10, R9.2
- new net SIM_CLK: IC5.32, R22.1
- new net SIM_DATA: C19.2, IC5.31, R24.1
- new net SIM_RST: IC5.33, R23.1
- new net SIM_VDD: C20.2, IC5.30, J6.1, Z2.2
- new net SPK+: IC5.21
- new net SPK-: IC5.22
- new net STATUS_LED: IC5.66
- new net TXD: IC5.9, R8.2
- net AUDIO_GND: no longer S5.42
- net DSR0: now also IC5.6; no longer S5.34, S5.35
- net GND: now also C18.1, C19.1, C20.1, C21.1, IC5.17, IC5.18, IC5.29, IC5.39, IC5.45, IC5.46, IC5.53, IC5.54, IC5.58, IC5.59, IC5.61, IC5.62, IC5.63, IC5.64, IC5.65, J6.6, Q4.2, R25.1, U$9.-, Y1.2, Z1.3, Z2.3; no longer C2.1, C3.1, Q3.2, S5.21, S5.22, S5.23, S5.24, S5.25, S5.6
- net GSM_READY: no longer S5.5
- net N$15: now also IC1.8, Y1.3; no longer Q3.1, R18.1
- net N$18: now also IC5.1, R6.2; no longer S5.44, SJ3.2, SJ6.2
- net N$19: now also Q4.3, R6.1; no longer JP13.2, S4.1, S5.50, SJ6.1
- net N$9: now also IC1.7, Y1.1; no longer S4.2A, S4.2B, S5.43, SJ2.2
- net NET_OK: no longer S5.13
- net ON_KEY: now also R26.2; no longer S5.41
- net SENSE_1V8: no longer Q3.3
- net VCC: now also C21.2, IC5.55, IC5.56, IC5.57; no longer S5.26, S5.27, S5.28, S5.29, S5.30
Routing:
- net N$19: track 62.6 -> 0.00 mm, vias 1 -> 0
- net EARN: track 0.00 -> 57.9 mm, vias 0 -> 1
- net N$20: track 55.7 -> 0.00 mm
- net EARP: track 0.00 -> 48.4 mm
- net N$26: track 47.4 -> 0.00 mm, vias 3 -> 0
- net N$18: track 42.8 -> 0.00 mm, vias 2 -> 0
- net N$9: track 46.1 -> 6.98 mm, vias 1 -> 0
- net N$22: track 38.4 -> 0.00 mm, vias 2 -> 0
- net ON_KEY: track 39.2 -> 0.76 mm, vias 2 -> 0
- net VCC: track 138.8 -> 173.2 mm
- net MIC1P: track 0.00 -> 31.4 mm, vias 0 -> 1
- net MIC1N: track 0.00 -> 28.4 mm, vias 0 -> 2
- net SENSE_1V8: track 19.3 -> 0.00 mm
- net XTL1: track 16.8 -> 0.00 mm
- net GND: track 48.7 -> 32.0 mm
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Other:
- board text added: "ArduPhone2"
- board text added: "v2.0"
- board text added: "www.freetronics.com/phone2"
