File: PHONE2.sch (EAGLE design)
At the start: 106 parts, among them IC1 ATMEGA1284P, IC2 FT230X, IC3 LTC4054, IC4 LP2985-33DBVR, J1 Power, J2 Analog, J3 Digital_8_13, J4 Digital_0_7, P1 USB-6PSMT, P2 ICSP:MAIN, Q1 2N7002 SOT-23, Q2 2N7002, Q3 BC846ALTIG, SW0 0, SW1 1, SW10 *, SW11 #, SW12 LEFT, SW13 DOWN, SW14 RIGHT, SW15 UP, SW2 2, SW3 3, SW4 4, SW5 5, SW6 6, SW7 7, SW8 8, SW9 9, X1 8MHz

Commit message: Routing and schematic work
Parts:
- removed C2, C3: 22pF 0603, freetronics-master-v1.1:CAP0603
- removed Q3: BC846ALTIG, freetronics-original:TRANSISTOR_NPNSOT23-3
- removed R18: 10K 0603, freetronics-master-v1.1:RESISTOR0603
- removed S5: Hirose DF12C(3.0)-50DP-0.5V, freetronics-jon:ADH8066
- removed TP3, TP4, TP5: TEST-POINT, freetronics-original:TEST-POINT2
- removed X1: 8MHz, freetronics-master-v1:CRYSTALHC49UV
- added C18, C20, C21: 100nF, freetronics-master-v1:CAP0603
- added C19: 22pF, freetronics-master-v1:CAP0603
- added IC5: SIM900, ICs_v54:SIM900
- added J6: SIM Socket, SparkFun2:SIMHOLDER3
- added Q4: 2N7002, freetronics-luke:2N7002
- added R22, R23, R24: 22R, freetronics-master-v1:RESISTOR0603
- added R25: 100K, freetronics-master-v1:RESISTOR0603
- added R26: 10R, freetronics-master-v1:RESISTOR0603
- added U$9: XH414H-IV01E, cellphone:SUPERCAPPAS
- added Y1: RESONATORSMD, SparkFun:RESONATORSMD
- added Z1, Z2: PGB102ST23, freetronics-luke:PGB102ST23
- R6: value 1M 0603 -> 100K; device freetronics-master-v1.1:RESISTOR0603 -> freetronics-master-v1:RESISTOR0603; PACKAGE (none) -> 0603
- TP1, TP2: value TEST-POINT -> TEST-POINT2
Connections:
- removed net N$20: JP13.1, S4.3, S4.4, S5.EARP
- removed net N$21: R8.2, S5.TXD0
- removed net N$22: R9.2, S5.RXD0
- removed net N$23: S5.VCHARGE18, TP3.1
- removed net N$24: S5.VCHARGE19, TP4.1
- removed net N$25: S5.CHV_DRV, TP5.1
- removed net N$26: R18.2, S5.1V8_OUT
- removed net N$30: S5.ADC1, TP1.1
- removed net N$31: S5.ADC2_BATTEMP, TP2.1
- removed net XTL1: C3.2, IC1.XTAL1, R6.1, X1.1
- removed net XTL2: C2.2, IC1.XTAL2, R6.2, X1.2
- new net !GSM_RESET: C18.2, IC5.NRESET
- new net CTS: IC5.CTS
- new net DBG_RXD: IC5.DBG_RXD, TP1.1
- new net DBG_TXD: IC5.DBG_TXD, TP2.1
- new net DCD: IC5.DCD
- new net DISP_CLK: IC5.DISP_CLK
- new net DISP_CS: IC5.DISP_CS
- new net DISP_DATA: IC5.DISP_DATA
- new net DISP_DC: IC5.DISP_D/C
- new net EARN: JP13.2, S4.1, SJ6.1
- new net EARP: JP13.1, S4.3, S4.4
- new net MIC+: IC5.MIC_P
- new net MIC-: IC5.MIC_N
- new net MIC1N: SJ3.2, SJ6.2
- new net MIC1P: S4.2A, S4.2B, SJ2.2
- new net N$28: J6.RST, R23.2, Z2.P$1
- new net N$29: IC5.VRTC, U$9.+
- new net N$40: J6.CLK, R22.2, Z1.P$1
- new net N$49: J6.I/O, R24.2, Z1.P$2
- new net N$69: Q4.G, R25.2, R26.1
- new net NETWORK_LED: IC5.NETLIGHT
- new net RF_ANT: IC5.RF_ANT
- new net RI: IC5.RI
- new net RTS: IC5.RTS
- new net RXD: IC5.RXD, R9.2
- new net SIM_CLK: IC5.SIM_CLK, R22.1
- new net SIM_DATA: C19.2, IC5.SIM_DATA, R24.1
- new net SIM_RST: IC5.SIM_RST, R23.1
- new net SIM_VDD: C20.2, IC5.SIM_VDD, J6.VCC, Z2.P$2
- new net SPK+: IC5.SPK_P
- new net SPK-: IC5.SPK_N
- new net STATUS_LED: IC5.STATUS
- new net TXD: IC5.TXD, R8.2
- net AUDIO_GND: no longer S5.GND@42
- net DSR0: now also IC5.DSR; no longer S5.CTS0, S5.DSR0
- net GND: now also C18.1, C19.1, C20.1, C21.1, IC5.GND@0, IC5.GND@1, IC5.GND@10, IC5.GND@11, IC5.GND@12, IC5.GND@13, IC5.GND@14, IC5.GND@2, IC5.GND@3, IC5.GND@4, IC5.GND@5, IC5.GND@6, IC5.GND@7, IC5.GND@8, IC5.GND@9, J6.GND, Q4.S, R25.1, U$9.-, Y1.2, Z1.P$3, Z2.P$3; no longer C2.1, C3.1, Q3.E, S5.GND@21, S5.GND@22, S5.GND@23, S5.GND@24, S5.GND@25, S5.GND@6
- net GSM_READY: no longer S5.GPIO10_READY
- net N$15: now also IC1.XTAL1, Y1.3; no longer Q3.B, R18.1
- net N$18: now also IC5.PWRKEY, R6.2; no longer S5.MIC1_N, SJ3.2, SJ6.2
- net N$19: now also Q4.D, R6.1; no longer JP13.2, S4.1, S5.EARN, SJ6.1
- net N$9: now also IC1.XTAL2, Y1.1; no longer S4.2A, S4.2B, S5.MIC1_P, SJ2.2
- net NET_OK: no longer S5.GPIO3_GSM_NET_OK
- net ON_KEY: now also R26.2; no longer S5.ON_KEY
- net SENSE_1V8: no longer Q3.C
- net VCC: now also C21.2, IC5.VBAT@0, IC5.VBAT@1, IC5.VBAT@2; no longer S5.VBAT@26, S5.VBAT@27, S5.VBAT@28, S5.VBAT@29, S5.VBAT@30
Other:
- note added: "(C)2014 Freetronics Pty Ltd"
- note added: "SKU: PHONE2"
- note added: "TODO: Antenna mount Power switch xh414h-iv01e RTC battery Serial level shifters"
- note added: "V2.0 (2014-03-18)"
- note added: "www.freetronics.com/phone2"
- note removed: "(C)2013 Freetronics Pty Ltd"
- note removed: "ADH8066"
- note removed: "SKU: PHONE"
- note removed: "TODO: Antenna mount Power switch"
- note removed: "V1.2 (2013-11-26)"
- note removed: "www.freetronics.com/phone"
- moved on the sheet: C10, C6, R6, TP1, TP2
